Commit message: push version that loads to mj viewer

File: urdf/lite6.urdf (robot description, URDF)
Before this commit: robot ufactory_lite6, 9 links, 8 joints
Links:
- link link_base: geometry collision mesh filename=../meshes/lite6/collision/base.stl; visual mesh filename=../meshes/lite6/visual/base.stl
